File: final_kicad/final_kicad_bk/_autosave-final_kicad.kicad_sch (KiCad schematic)
At the start: 36 parts, among them J3 Reflectance Sensor Array, M1 Motor, M3 Servo for Side Indicator, M4 Motor_Servo, Q1 Photo_NPN, SW1 Reset, U1 SN754410, U2 MCP6294, U2 PIC32MX170F256B, U4 Comparator

Commit message: update
Parts:
- added C8: 0.1uF, symbol ME218_BaseLib:Cap
- added D10: Jumbo LED Indicator, symbol ME218_BaseLib:LED
- added D9: Jumbo LED Indicators, symbol ME218_BaseLib:LED
- added PRG2: MPLAB_Snap, symbol ME218_BaseLib:MPLAB_Snap
- added Q2: MOSFET-N, symbol ME218_BaseLib:MOSFET-N
- added R10, R_limit, R_pull: 10k, symbol ME218_BaseLib:Res1
- added R9: 1k, symbol ME218_BaseLib:Res1
- added SW2: Reset, symbol ME218_BaseLib:SW_Push
- M4: value Motor_Servo -> Servo for Gripper
Connections:
- net +3.3V: now also PRG2.2 (Vdd), Q2.1 (D), R10.2
- net GND: now also PRG2.3 (Vss)
- net GNDREF: now also C8.2, D10.1 (K), D9.1 (K), R_pull.2, SW2.2
- net tera: now also U2.15 (PGEC3/5VT/RB6), U2.16 (5VT/RB7)
- net at PRG1.1 (~{MCLR}/Vpp), R1.1: now also U2.1 (~{MCLR})
- net at U2.1 (~{MCLR}): now also PRG2.1 (~{MCLR}/Vpp), R9.1
- net at U2.10 (RA3): now also Q2.2 (G), R_pull.1
- net at U2.4 (PGED1/RB0): now also PRG2.4 (PGData)
- net at U2.5 (PGEC1/RB1): now also PRG2.5 (PGClk)
- net at U2.9 (RA2): now also M4.1 (PWM)
- net at U1.2 (1A): now also U2.22 (RB11); no longer U2.6 (RB2)
- net at U2.26 (RB15): now also J3.5 (Pin_5)
- net at J3.6 (Pin_6): now also U2.6 (RB2)
- new net: C8.1, R10.1, R9.2, SW2.1
- new net: D10.2 (A), D9.2 (A), R_limit.2
- new net: Q2.3 (S), R_limit.1
Other:
- moved on the sheet: M4
