File: final_kicad/final_kicad_bk/final_kicad.kicad_sch (KiCad schematic)
At the start: 70 parts, among them J3 Reflectance Sensor Array, M1 Motor, M3 Servo for Side Indicator, M4 Servo for Gripper, M5 Motor_Step_4Wire, M6 Motor for Linear Actuator, Q1 Photo_NPN, Q2 MOSFET-N, SW1 Reset, SW2 Reset, U0 PIC32MX170F256B, U1 SN754410, U2 MCP6294, U2 PIC32MX170F256B, U4 Comparator, U5 L293NE, U6 L293NE

Commit message: clean kicad
Parts:
- renumbered U0 to U2
Connections:
- net +3.3V: now also J3.1 (Pin_1)
- net +5V: no longer U6.1 (EN1,2)
- net Earth: now also J3.2 (Pin_2)
- net GND: no longer U6.9 (EN3,4)
- net at U2.26 (RB15): no longer M3.1 (PWM)
- net at U2.2 (RA0): now also J3.7 (Pin_7); no longer J3.1 (Pin_1)
- net at U2.3 (RA1): now also J3.8 (Pin_8); no longer J3.2 (Pin_2)
- net at U2.9 (RA2): now also M3.1 (PWM)
Other:
- note added: "For Robot Arm"
- note removed: "For Linear Stage"

Commit message: clean kicad
Parts:
- renumbered U2 to U0
Connections:
- net +3.3V: no longer J3.1 (Pin_1)
- net +5V: now also U6.1 (EN1,2)
- net Earth: no longer J3.2 (Pin_2)
- net GND: now also U6.9 (EN3,4)
- net MISO/SDI: now also U0.24 (RB13); no longer U0.14 (PGED3/5VT/RB5)
- net at M4.1 (PWM): now also U0.14 (PGED3/5VT/RB5); no longer U0.24 (RB13)
- net at U0.26 (RB15): now also M3.1 (PWM)
- net at U2.2 (RA0): now also J3.1 (Pin_1); no longer J3.7 (Pin_7)
- net at U2.3 (RA1): now also J3.2 (Pin_2); no longer J3.8 (Pin_8)
- net at U2.9 (RA2): no longer M3.1 (PWM)
Other:
- note added: "For Linear Stage"
- note removed: "For Robot Arm"
