File: final_kicad/final_kicad_bk/final_kicad.kicad_sch (KiCad schematic)
At the start: 70 parts, among them J3 Reflectance Sensor Array, M1 Motor, M3 Servo for Side Indicator, M4 Servo for Gripper, M5 Motor_Step_4Wire, M6 Motor for Linear Actuator, Q1 Photo_NPN, Q2 MOSFET-N, SW1 Reset, SW2 Reset, U0 PIC32MX170F256B, U1 SN754410, U2 MCP6294, U2 PIC32MX170F256B, U4 Comparator, U5 L293NE, U6 L293NE

Commit message: refine kicad
Parts:
- renumbered U0 to PIC0
Connections:
- net +6V: now also D15.2 (A), D16.1 (K), M5.2 (-), R12.1, U5.6 (2Y)
- net BEACON_SENSOR: now also U2.22 (RB11); no longer U2.10 (RA3)
- net DO: now also PIC0.10 (RA3); no longer PIC0.6 (RB2)
- net MISO/SDI: now also PIC0.14 (PGED3/5VT/RB5); no longer PIC0.24 (RB13)
- net MOSI/SDI: now also U2.9 (RA2); no longer U2.14 (PGED3/5VT/RB5)
- net OC1: now also U2.25 (RB14); no longer U2.7 (RB3)
- net SCK: now also U2.26 (RB15); no longer U2.25 (RB14)
- net at Q2.2 (G), R_pull.1: now also PIC0.12 (RA4); no longer PIC0.10 (RA3)
- net at M4.1 (PWM): now also PIC0.26 (RB15); no longer PIC0.14 (PGED3/5VT/RB5)
- net at M3.1 (PWM): now also PIC0.24 (RB13); no longer PIC0.26 (RB15)
- net at U1.2 (1A): now also U2.14 (PGED3/5VT/RB5); no longer U2.22 (RB11)
- net at J3.5 (Pin_5): now also U2.7 (RB3); no longer U2.26 (RB15)
Other:
- moved on the sheet: C1, C2, C3, C4, C5, C6, C7, C8, C9, D1, D2, D5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
