File: final_kicad/final_kicad.kicad_sch (KiCad schematic)
At the start: 70 parts, among them J3 Reflectance Sensor Array, M1 Motor, M3 Servo for Side Indicator, M4 Servo for Gripper, M5 Motor_Step_4Wire, M6 Motor for Linear Actuator, Q1 Photo_NPN, Q2 MOSFET-N, SW1 Reset, SW2 Reset, U1 SN754410, U2 MCP6294, U2 PIC32MX170F256B, U4 Comparator, U5 L293NE, U6 L293NE

Commit message: refine planner
Connections:
- net BEACON_SENSOR: now also PIC0.9 (RA2); no longer U2.22 (RB11)
Other:
- moved on the sheet: Q1, R3, R4, R5, R6, R7, R8, U2A, U4A
