File: final_kicad/final_kicad.kicad_sch (KiCad schematic)
At the start: 70 parts, among them J3 Reflectance Sensor Array, M1 Motor, M3 Servo for Side Indicator, M4 Servo for Gripper, M5 Motor_Step_4Wire, M6 Motor for Linear Actuator, Q1 Photo_NPN, Q2 MOSFET-N, SW1 Reset, SW2 Reset, U1 SN754410, U2 MCP6294, U2 PIC32MX170F256B, U4 Comparator, U5 L293NE, U6 L293NE

Commit message: kicad update
Connections:
- net OC1: now also U2.12 (RA4); no longer U2.25 (RB14)
Changed lines of the file:
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@@
     (stroke (width 0) (type default))
   )
-  (wire (pts (xy 382.27 271.78) (xy 382.27 302.26))
+  (wire (pts (xy 382.27 271.78) (xy 382.27 327.66))
     (stroke (width 0) (type default))
   )
@@
     (stroke (width 0) (type default))
   )
-  (wire (pts (xy 382.27 302.26) (xy 363.22 302.26))
-    (stroke (width 0) (type default))
-  )
   (wire (pts (xy 25.4 129.54) (xy 30.48 129.54))
     (stroke (width 0) (type default))
@@
     (stroke (width 0) (type default))
   )
+  (wire (pts (xy 313.69 285.75) (xy 323.85 285.75))
+    (stroke (width 0) (type default))
+  )
   (wire (pts (xy 274.32 119.38) (xy 274.32 114.3))
     (stroke (width 0) (type default))
@@
     (stroke (width 0) (type default))
   )
+  (wire (pts (xy 313.69 327.66) (xy 313.69 285.75))
+    (stroke (width 0) (type default))
+  )
   (wire (pts (xy 243.84 116.84) (xy 246.38 116.84))
     (stroke (width 0) (type default))
@@
     (stroke (width 0) (type default))
   )
+  (wire (pts (xy 382.27 327.66) (xy 313.69 327.66))
+    (stroke (width 0) (type default))
+  )
